File: board/atmega.sch (KiCad schematic (older format))
At the start: 21 parts, among them J1.1 Conn_01x04, J1.2 Conn_01x06, J1.3 Conn_01x16, J1.4 Conn_01x11, J1.5 Conn_01x13, J1.6 Conn_01x11, SW1 SW_Push, U101 ATmega128A-AU, X101 Crystal

Commit message: updated pcb design
Parts:
- added D1.2, D1.3, D1.4, D1.5: LED, LED_SMD:LED_0805_2012Metric_Pad1.15x1.40mm_HandSolder, symbol Device:LED
- added J1.11: EN, TestPoint:TestPoint_THTPad_1.0x1.0mm_Drill0.5mm, symbol Connector_Generic:Conn_01x01
- added J1.12: ALED, TestPoint:TestPoint_THTPad_1.0x1.0mm_Drill0.5mm, symbol Connector_Generic:Conn_01x01
- added J1.13: STAT, TestPoint:TestPoint_THTPad_1.0x1.0mm_Drill0.5mm, symbol Connector_Generic:Conn_01x01
- added J1.14: SELECT, TestPoint:TestPoint_THTPad_1.0x1.0mm_Drill0.5mm, symbol Connector_Generic:Conn_01x01
- added J1.15, J1.16, J1.17, J1.18, J1.19, J1.20, J1.21, J1.22, J1.26, J1.28, J1.29, J1.30, J1.31: (no value), TestPoint:TestPoint_THTPad_1.0x1.0mm_Drill0.5mm, symbol Connector_Generic:Conn_01x01
- added J1.23: GND, TestPoint:TestPoint_THTPad_1.0x1.0mm_Drill0.5mm, symbol Connector_Generic:Conn_01x01
- added J1.24: VCC, TestPoint:TestPoint_THTPad_1.0x1.0mm_Drill0.5mm, symbol Connector_Generic:Conn_01x01
- added J1.25: RST, TestPoint:TestPoint_THTPad_1.0x1.0mm_Drill0.5mm, symbol Connector_Generic:Conn_01x01
- added J1.27: SWI, TestPoint:TestPoint_THTPad_1.0x1.0mm_Drill0.5mm, symbol Connector_Generic:Conn_01x01
- added J1.32: RTS, TestPoint:TestPoint_THTPad_1.0x1.0mm_Drill0.5mm, symbol Connector_Generic:Conn_01x01
- added J1.33: CTS, TestPoint:TestPoint_THTPad_1.0x1.0mm_Drill0.5mm, symbol Connector_Generic:Conn_01x01
- added J1.34: RXD, TestPoint:TestPoint_THTPad_1.0x1.0mm_Drill0.5mm, symbol Connector_Generic:Conn_01x01
- added J1.35: TXD, TestPoint:TestPoint_THTPad_1.0x1.0mm_Drill0.5mm, symbol Connector_Generic:Conn_01x01
- added J1.36, J1.7: Conn_01x04, Connector_PinHeader_2.54mm:PinHeader_1x04_P2.54mm_Vertical, symbol Connector_Generic:Conn_01x04
- added J37: Conn_01x05, Connector_PinHeader_2.54mm:PinHeader_1x05_P2.54mm_Vertical, symbol Connector_Generic:Conn_01x05
- added JP1.1, JP1.2, JP1.3, JP1.4: M4PWM, Jumper:SolderJumper-2_P1.3mm_Open_TrianglePad1.0x1.5mm, symbol Jumper:Jumper_2_Open
- added Q1.1: AO3400A, Package_TO_SOT_SMD:SOT-23, symbol Transistor_FET:AO3400A
- added R1.10, R1.11, R1.12, R1.13, R1.14, R1.4, R1.5, R1.6, R1.7, R1.8, R1.9: R, Resistor_SMD:R_0805_2012Metric_Pad1.20x1.40mm_HandSolder, symbol Device:R
- added SW1.2, SW1.3: SW_Push, Button_Switch_THT:SW_PUSH_6mm_H4.3mm, symbol Switch:SW_Push
Connections:
- net labels added: 3.3V, B_RXD, B_STAT, B_TXD, M1A, M1B, M2A, M2B, M2PWM, M3A, M3B, M3PWM, M4A, M4B, M4PWM
- net labels removed: PWM2, PWM3, PWM4, PWM5, PWM6, PWM7
- wire segments 163 -> 282
