File: board/drv8825.sch (KiCad schematic (older format))
At the start: 11 parts, among them J2.1 Conn_01x02, J2.2 Conn_01x02, J2.3 Conn_01x02, J2.4 Conn_01x02

Commit message: updated pcb design
Parts:
- added H5, H6, H7: MountingHole, MountingHole:MountingHole_2.5mm_Pad, symbol Mechanical:MountingHole
- added J2.5, J2.6, J2.7, J2.8: Conn_01x04, Connector_PinHeader_2.54mm:PinHeader_1x04_P2.54mm_Vertical, symbol Connector_Generic:Conn_01x04
- added TP1, TP10, TP100, TP101, TP102, TP11, TP12, TP13, TP14, TP15, TP16, TP17, TP18, TP19, TP2, TP20, TP21, TP22, TP23, TP24, TP25, TP26, TP27, TP28, TP29, TP3, TP30, TP31, TP32, TP33, TP34, TP35, TP36, TP37, TP38, TP39, TP4, TP40, TP41, TP42, TP43, TP44, TP45, TP46, TP47, TP48, TP49, TP5, TP50, TP51, TP52, TP53, TP54, TP55, TP56, TP57, TP58, TP59, TP6, TP60, TP61, TP62, TP63, TP64, TP65, TP66, TP67, TP68, TP69, TP7, TP70, TP71, TP72, TP73, TP74, TP75, TP76, TP77, TP78, TP79, TP8, TP80, TP81, TP82, TP83, TP84, TP85, TP86, TP87, TP88, TP89, TP9, TP90, TP91, TP92, TP93, TP94, TP95, TP96, TP97, TP98, TP99: TestPoint, TestPoint:TestPoint_Pad_4.0x4.0mm, symbol Connector:TestPoint
- added U99: viking, board:viking, symbol custom:viking
Connections:
- wire segments 19 -> 29
